File: src/mael/eagle/mael.sch (EAGLE design)
At the start: 12 parts

Commit message: Finish up mael motor PCB
Parts:
- removed 3V, 5V: (no value), SparkFun-Connectors:BATTERY_CONN_DEANS
- added 12V1: (no value), SparkFun-Connectors:BATTERY_CONN_DEANS
- added C1, C2, C3, C4: (no value), rcl:C-EU050-024X044
- added IC1, IC2: (no value), v-reg:78XXL
Connections:
- net +12V: now also 12V1.+, C2.2, C4.2, IC1.IN, IC2.IN
- net +3V3: now also C3.2, IC1.OUT; no longer 3V.+
- net +5V: now also C1.2, IC2.OUT; no longer 5V.+
- net GND: now also 12V1.-, C1.1, C2.1, C3.1, C4.1; no longer 3V.-, 5V.-
Other:
- moved on the sheet: 12V
